Commit message: handle urdf files with a manager containing one single object (no joints)

File: python/bullet/samples/data/box.urdf (robot description, URDF)
Before this commit: robot box, 1 links, 0 joints
Links:
- link boxLink: mass .0 -> 10

Commit message: display all shapes of a multi object. Doesn t work well ...

File: python/bullet/samples/data/box.urdf (robot description, URDF)
Before this commit: robot box, 1 links, 0 joints
Links:
- removed link boxLink
- added link base_link, mass 10; collision mesh filename=box-T2F_N3F_V3F.obj scale=1 1 1; visual mesh filename=box-T2F_N3F_V3F.obj scale=1 1 1
- added link right_leg, mass 10; collision mesh filename=box-T2F_N3F_V3F.obj scale=1 1 1; visual mesh filename=box-T2F_N3F_V3F.obj scale=1 1 1
Joints:
- added joint base_to_right_leg: type fixed, parent base_link, child right_leg, origin xyz=1 0 0
