Commit message: Motor applied on a joint with key up and key down

File: python/bullet/samples/data/006-box.urdf (robot description, URDF)
Before this commit: robot box, 2 links, 1 joints
Joints:
- joint base_to_right_leg: limit lower=-1.57 upper=1.57 effort=1000.0 velocity=0.5 -> lower=-1.57 upper=1.57 effort=1000.0 velocity=1000
