Commit message: start to build our humanoid

File: python/bullet/samples/data/007-humanoid.urdf (robot description, URDF)
Before this commit: robot box, 2 links, 1 joints
Links:
- removed link right_leg
- added link pelvis_pitch, mass 2; collision mesh filename=box-T2F_N3F_V3F.obj scale=1 1 1; visual mesh filename=box-T2F_N3F_V3F.obj scale=1 1 1
Joints:
- joint base_to_right_leg: axis 0 1 0 -> 0 0 0.5
