Commit message: add maze game from 18th Raspberry Inside magazine

File: python/bullet/samples/data/008-multi-shape.urdf (robot description, URDF)
Before this commit: robot box, 4 links, 3 joints
Links:
- removed link left_leg_top
- removed link right_leg_top
- added link left_leg_top_x_axis, mass 10; collision mesh filename=box-T2F_N3F_V3F.obj scale=0.5 0.5 0.25; visual mesh filename=box-T2F_N3F_V3F.obj scale=0.5 0.5 0.25
- added link left_leg_top_y_axis, mass 10; collision mesh filename=box-T2F_N3F_V3F.obj scale=0.5 0.5 0.25; visual mesh filename=box-T2F_N3F_V3F.obj scale=0.5 0.5 0.25
- added link right_leg_top_x_axis, mass 10; collision mesh filename=box-T2F_N3F_V3F.obj scale=0.5 0.5 0.25; visual mesh filename=box-T2F_N3F_V3F.obj scale=0.5 0.5 0.25
- added link right_leg_top_y_axis, mass 10; collision mesh filename=box-T2F_N3F_V3F.obj scale=0.5 0.5 0.25; visual mesh filename=box-T2F_N3F_V3F.obj scale=0.5 0.5 0.25
Joints:
- removed joint pelvis_to_left_leg_top
- removed joint pelvis_to_right_leg_top
- added joint left_leg_top_y_axis_to_left_leg_top_x_axis: type revolute, parent left_leg_top_y_axis, child left_leg_top_x_axis, origin xyz=0 0 -0.5 rpy=0 0 0, axis 1 0 0, limit lower=-0.785 upper=0.785 effort=1000.0 velocity=1000
- added joint pelvis_to_left_leg_top_y_axis: type revolute, parent pelvis, child left_leg_top_y_axis, origin xyz=1 0 -0.5 rpy=0 0 0, axis 0 1 0, limit lower=-1.57 upper=0.2 effort=1000.0 velocity=1000
- added joint pelvis_to_right_leg_top_y_axis: type revolute, parent pelvis, child right_leg_top_y_axis, origin xyz=-1 0 -0.5 rpy=0 0 0, axis 0 1 0, limit lower=-0.2 upper=1.57 effort=1000.0 velocity=1000
- added joint right_leg_top_y_axis_to_right_leg_top_x_axis: type revolute, parent right_leg_top_y_axis, child right_leg_top_x_axis, origin xyz=0 0 -0.5 rpy=0 0 0, axis 1 0 0, limit lower=-0.785 upper=0.785 effort=1000.0 velocity=1000
