Commit message: multi shape urdf start to look like at a humanoid + scale is now working properly

File: python/bullet/samples/data/r2d2/r2d2.urdf (robot description, URDF)
Before this commit: robot physics, 16 links, 15 joints
Links:
- link left_gripper: geometry collision mesh filename=l_finger.stl; visual mesh filename=l_finger.stl scale=0.5 0.6 0.7
